File: hw/eagle/main.brd (EAGLE design)
At the start: 49.2 x 49.5 mm, 12 parts

Commit message: [ add ] hw, wip
Parts:
- moved CON_REED 40.6 mm to (47.0, 8.89), turned to 270 degrees
- moved C1 39.7 mm to (8.89, 27.9)
- moved C2 38.7 mm to (8.89, 24.1)
- moved JMP_VCC_COIN_OR_ALT 33.2 mm to (6.35, 14.0)
- moved PCB1 31.7 mm to (41.9, 2.54), turned to 90 degrees
- moved CON_NRF 28.7 mm to (11.4, 5.08), turned to 180 degrees
- moved CON_COIN_HOLDER 25.7 mm to (11.4, 19.1)
- moved CON_VCC_SWITCH 21.6 mm to (5.08, 19.1)
- moved CON_GND 21.6 mm to (15.2, 44.5)
- moved R1 16.6 mm to (19.1, 19.1)
- moved CON_VCC_EN 16.5 mm to (15.2, 40.6)
- moved CON_IO 5.68 mm to (15.2, 36.8), turned to 180 degrees
Routing:
- added copper zone on layer 1, net GND

Commit message: [ add ] main.bom
Parts:
- removed C2: 330u, rcl:C1206K
- added C3: 330u, rcl:PANASONIC_F
- CON_COIN_HOLDER, CON_REED, CON_VCC_SWITCH: device pinhead:1X02 -> SparkFun:1X02
- CON_GND, CON_IO, CON_VCC_EN: device con-lstb:MA05-1 -> SparkFun:1X05
- JMP_VCC_COIN_OR_ALT: device con-lstb:MA03-1 -> SparkFun:1X03
- R1: value 470K -> 1M
- moved JMP_VCC_COIN_OR_ALT 32.1 mm to (36.8, 3.81)
- moved C1 26.2 mm to (19.1, 3.81)
- moved CON_COIN_HOLDER 24.4 mm to (30.5, 3.81)
- moved CON_VCC_SWITCH 24.4 mm to (24.1, 3.81)
- moved R1 18.1 mm to (33.0, 30.5), turned to 180 degrees
- moved CON_VCC_EN 8.52 mm to (7.62, 44.5)
- moved CON_GND 8.03 mm to (7.62, 47.0)
- moved PCB1 6.48 mm to (43.2, 8.89)
- moved CON_NRF 6.35 mm to (11.4, 11.4)
- moved CON_IO 5.68 mm to (17.8, 41.9)
- moved CON_REED 3.81 mm to (47.0, 12.7)
Connections:
- net COIN_VCC: now also C3.+; no longer C2.1
- net GND: now also C3.-; no longer C2.2

Commit message: [ update ] route, wip
Parts:
- moved CON_COIN_HOLDER 25.7 mm to (8.89, 17.8)
- moved R1 5.24 mm to (31.8, 25.4)
- moved PCB1 1.27 mm to (41.9, 8.89)
Routing:
- net POW_VCC_EN: track 0.00 -> 74.5 mm
- net UC_PORTC0: track 0.00 -> 52.1 mm
- net UC_PORTC1: track 0.00 -> 47.0 mm
- net NRF_SCK: track 0.00 -> 44.5 mm
- net UC_PORTC2: track 0.00 -> 41.9 mm
- net REED_EN: track 0.00 -> 36.8 mm
- net UC_PORTC3: track 0.00 -> 36.8 mm
- net NRF_TXEN: track 0.00 -> 31.8 mm
- net NRF_MISO: track 0.00 -> 31.8 mm
- net NRF_CSN: track 0.00 -> 31.7 mm
- net NRF_PWR: track 0.00 -> 21.6 mm
Other:
- board text added: "FLM designs"
- board text added: "bano_reed_v0000"

Commit message: [ update ] route, wip
Parts:
- removed CON_GND, CON_IO, CON_VCC_EN: (no value), SparkFun:1X05
- removed CON_NRF: (no value), con-lstb:MA07-2
- removed CON_VCC_SWITCH: (no value), SparkFun:1X02
- removed JMP_VCC_COIN_OR_ALT: (no value), SparkFun:1X03
- added COIN_OR_ALT: (no value), SparkFun:1X03
- added GND, IO, VCC: (no value), SparkFun:1X04
- added NRF: (no value), con-lstb:MA07-2
- added VCC_SWITCH: (no value), SparkFun:1X02
- CON_COIN_HOLDER: device SparkFun:1X02 -> SparkFun:BATTCOM_20MM_PTH
- moved C3 40.7 mm to (12.7, 44.5), turned to 180 degrees
- moved C1 39.9 mm to (3.81, 40.6)
- moved R1 5.24 mm to (30.5, 20.3)
- moved PCB1 5.08 mm to (41.9, 3.81)
- moved CON_COIN_HOLDER 4.58 mm to (11.4, 14.0), flipped to the bottom, turned to 90 degrees
- renumbered CON_REED to REED
Connections:
- removed net N$9: CON_GND.2
- removed net UC_PORTB1: CON_IO.5, PCB1.9
- net ALT_VCC: now also COIN_OR_ALT.1; no longer JMP_VCC_COIN_OR_ALT.1
- net COIN_VCC: now also COIN_OR_ALT.3; no longer JMP_VCC_COIN_OR_ALT.3
- net GND: now also GND.1, GND.2, GND.3, GND.4, NRF.1, NRF.2; no longer CON_GND.1, CON_GND.3, CON_GND.4, CON_GND.5, CON_NRF.1, CON_NRF.2
- net NRF_AM: now also NRF.8; no longer CON_NRF.8
- net NRF_CD: now also NRF.9; no longer CON_NRF.9
- net NRF_CE: now also NRF.12; no longer CON_NRF.12
- net NRF_CSN: now also NRF.3; no longer CON_NRF.3
- net NRF_DR: now also NRF.7; no longer CON_NRF.7
- net NRF_MISO: now also NRF.6; no longer CON_NRF.6
- net NRF_MOSI: now also NRF.5; no longer CON_NRF.5
- net NRF_PWR: now also NRF.11; no longer CON_NRF.11
- net NRF_SCK: now also NRF.4; no longer CON_NRF.4
- net NRF_TXEN: now also NRF.13; no longer CON_NRF.13
- net NRF_UCK: now also NRF.10; no longer CON_NRF.10
- net POW_VCC: now also COIN_OR_ALT.2, VCC_SWITCH.1; no longer CON_VCC_SWITCH.1, JMP_VCC_COIN_OR_ALT.2
- net POW_VCC_EN: now also NRF.14, VCC.1, VCC.2, VCC.3, VCC.4, VCC_SWITCH.2; no longer CON_NRF.14, CON_VCC_EN.1, CON_VCC_EN.2, CON_VCC_EN.3, CON_VCC_EN.4, CON_VCC_EN.5, CON_VCC_SWITCH.2
- net UC_PORTC0: now also IO.4; no longer CON_IO.4
- net UC_PORTC1: now also IO.3; no longer CON_IO.3
- net UC_PORTC2: now also IO.2; no longer CON_IO.2
- net UC_PORTC3: now also IO.1; no longer CON_IO.1
Routing:
- net POW_VCC_EN: track 74.5 -> 130.8 mm
- net NRF_MOSI: track 0.00 -> 29.2 mm, vias 0 -> 1
- net NRF_DR: track 0.00 -> 29.2 mm
- net NRF_CE: track 0.00 -> 29.2 mm
- net NRF_CD: track 0.00 -> 26.7 mm, vias 0 -> 2
- net NRF_AM: track 0.00 -> 24.1 mm
- net UC_PORTC2: track 41.9 -> 24.7 mm
- net UC_PORTC1: track 47.0 -> 29.7 mm
- net UC_PORTC0: track 52.1 -> 34.8 mm
- net UC_PORTC3: track 36.8 -> 19.6 mm
- net REED_EN: track 36.8 -> 31.8 mm
