File: hw/eagle/main.sch (EAGLE design)
At the start: 10 parts

Commit message: [ update ] schematics progress
Parts:
- added C2: 330u, rcl:C-EUC1206K
- added CON_COIN_HOLDER: (no value), pinhead:PINHD-1X2
Connections:
- net COIN_VCC: now also C1.1, C2.1, CON_COIN_HOLDER.1
- net GND: now also C1.2, C2.2, CON_COIN_HOLDER.2
Other:
- note added: "bano_reed_v0000"
- note added: "https://github.com/texane/bano_reed"
- note added: "texane@gmail.com"
- note removed: "TODO: coin, connect to COIN_VCC"
- moved on the sheet: C1, CON_REED, CON_VCC_SWITCH, JMP_VCC_COIN_OR_ALT, R1
Changed lines of the file:
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@@
 <part name="CON_VCC_SWITCH" library="pinhead" deviceset="PINHD-1X2" device=""/>
 <part name="JMP_VCC_COIN_OR_ALT" library="con-lstb" deviceset="MA03-1" device=""/>
+<part name="CON_COIN_HOLDER" library="pinhead" deviceset="PINHD-1X2" device=""/>
+<part name="C2" library="rcl" deviceset="C-EU" device="C1206K" value="330u"/>
+<part name="FRAME1" library="frames" deviceset="A4L-LOC" device=""/>
 </parts>
 <sheets>
 <sheet>
 <plain>
-<text x="7.62" y="147.32" size="1.778" layer="91">TODO: coin, connect to COIN_VCC</text>
+<text x="66.04" y="5.08" size="1.6764" layer="94" font="vector">bano_reed_v0000</text>
+<text x="66.04" y="0" size="1.6764" layer="94" font="vector">https://github.com/texane/bano_reed</text>
+<text x="66.04" y="-5.08" size="1.6764" layer="94" font="vector">texane@gmail.com</text>
 </plain>
 <instances>
 <instance part="PCB1" gate="G$1" x="30.48" y="58.42" rot="R270"/>
 <instance part="CON_NRF" gate="G$1" x="109.22" y="55.88"/>
-<instance part="C1" gate="G$1" x="15.24" y="139.7"/>
-<instance part="R1" gate="G$1" x="-27.94" y="109.22"/>
-<instance part="CON_REED" gate="G$1" x="-15.24" y="109.22"/>
+<instance part="C1" gate="G$1" x="38.1" y="111.76" rot="MR0"/>
+<instance part="R1" gate="G$1" x="-33.02" y="106.68" rot="MR0"/>
+<instance part="CON_REED" gate="G$1" x="-45.72" y="106.68" smashed="yes" rot="MR0">
+<attribute name="NAME" x="-34.29" y="112.395" size="1.778" layer="95" rot="MR0"/>
+<attribute name="VALUE" x="-39.37" y="101.6" size="1.778" layer="96" rot="MR0"/>
+</instance>
 <instance part="CON_GND" gate="G$1" x="-45.72" y="40.64"/>
 <instance part="CON_VCC_EN" gate="G$1" x="-45.72" y="63.5"/>
 <instance part="CON_IO" gate="G$1" x="-45.72" y="86.36"/>
-<instance part="CON_VCC_SWITCH" gate="G$1" x="-15.24" y="124.46"/>
-<instance part="JMP_VCC_COIN_OR_ALT" gate="G$1" x="-45.72" y="142.24"/>
+<instance part="CON_VCC_SWITCH" gate="G$1" x="15.24" y="93.98" smashed="yes" rot="MR0">
+<attribute name="NAME" x="36.83" y="99.695" size="1.778" layer="95" rot="MR0"/>
+<attribute name="VALUE" x="21.59" y="88.9" size="1.778" layer="96" rot="MR0"/>
+</instance>
+<instance part="JMP_VCC_COIN_OR_ALT" gate="G$1" x="15.24" y="129.54"/>
+<instance part="CON_COIN_HOLDER" gate="G$1" x="15.24" y="111.76" smashed="yes" rot="MR0">
+<attribute name="NAME" x="36.83" y="117.475" size="1.778" layer="95" rot="MR0"/>
+<attribute name="VALUE" x="21.59" y="106.68" size="1.778" layer="96" rot="MR0"/>
+</instance>
+<instance part="C2" gate="G$1" x="30.48" y="111.76" rot="MR0"/>
+<instance part="FRAME1" gate="G$1" x="-99.06" y="-15.24" smashed="yes">
+<attribute name="DRAWING_NAME" x="118.11" y="0" size="2.54" layer="94" font="vector"/>
+<attribute name="LAST_DATE_TIME" x="118.11" y="-5.08" size="2.286" layer="94" font="vector"/>
+<attribute name="SHEET" x="131.445" y="-10.16" size="2.54" layer="94" font="vector"/>
+</instance>
 </instances>
 <busses>
@@
 <segment>
 <pinref part="R1" gate="G$1" pin="1"/>
-<wire x1="-33.02" y1="109.22" x2="-45.72" y2="109.22" width="0.1524" layer="91"/>
-<label x="-45.72" y="109.22" size="1.778" layer="95"/>
+<wire x1="-27.94" y1="106.68" x2="-15.24" y2="106.68" width="0.1524" layer="91"/>
+<label x="-15.24" y="106.68" size="1.778" layer="95" rot="MR0"/>
 </segment>
 <segment>
@@
 <label x="-35.56" y="35.56" size="1.778" layer="95"/>
 </segment>
+<segment>
+<pinref part="CON_COIN_HOLDER" gate="G$1" pin="2"/>
+<wire x1="17.78" y1="111.76" x2="17.78" y2="106.68" width="0.1524" layer="91"/>
+<wire x1="17.78" y1="106.68" x2="30.48" y2="106.68" width="0.1524" layer="91"/>
+<label x="48.26" y="106.68" size="1.778" layer="95" rot="MR0"/>
+<pinref part="C1" gate="G$1" pin="2"/>
+<wire x1="30.48" y1="106.68" x2="38.1" y2="106.68" width="0.1524" layer="91"/>
+<wire x1="38.1" y1="106.68" x2="48.26" y2="106.68" width="0.1524" layer="91"/>
+<junction x="38.1" y="106.68"/>
+<pinref part="C2" gate="G$1" pin="2"/>
+<junction x="30.48" y="106.68"/>
+</segment>
 </net>
 <net name="NRF_MISO" class="0">
@@
 <pinref part="CON_REED" gate="G$1" pin="2"/>
 <pinref part="R1" gate="G$1" pin="2"/>
-<wire x1="-17.78" y1="109.22" x2="-22.86" y2="109.22" width="0.1524" layer="91"/>
-<wire x1="-22.86" y1="109.22" x2="-22.86" y2="104.14" width="0.1524" layer="91"/>
-<junction x="-22.86" y="109.22"/>
-<wire x1="-22.86" y1="104.14" x2="-45.72" y2="104.14" width="0.1524" layer="91"/>
-<label x="-45.72" y="104.14" size="1.778" layer="95"/>
+<wire x1="-43.18" y1="106.68" x2="-38.1" y2="106.68" width="0.1524" layer="91"/>
+<wire x1="-38.1" y1="106.68" x2="-38.1" y2="101.6" width="0.1524" layer="91"/>
+<junction x="-38.1" y="106.68"/>
+<wire x1="-38.1" y1="101.6" x2="-15.24" y2="101.6" width="0.1524" layer="91"/>
+<label x="-15.24" y="101.6" size="1.778" layer="95" rot="MR0"/>
 </segment>
 <segment>
@@
 <segment>
 <pinref part="CON_VCC_SWITCH" gate="G$1" pin="1"/>
-<wire x1="-17.78" y1="127" x2="-45.72" y2="127" width="0.1524" layer="91"/>
-<label x="-45.72" y="127" size="1.778" layer="95"/>
+<wire x1="17.78" y1="96.52" x2="45.72" y2="96.52" width="0.1524" layer="91"/>
+<label x="45.72" y="96.52" size="1.778" layer="95" rot="MR0"/>
 </segment>
 <segment>
 <pinref part="JMP_VCC_COIN_OR_ALT" gate="G$1" pin="2"/>
-<wire x1="-38.1" y1="142.24" x2="-22.86" y2="142.24" width="0.1524" layer="91"/>
-<label x="-35.56" y="142.24" size="1.778" layer="95"/>
+<wire x1="22.86" y1="129.54" x2="38.1" y2="129.54" width="0.1524" layer="91"/>
+<label x="25.4" y="129.54" size="1.778" layer="95"/>
 </segment>
 </net>
@@
 <segment>
 <pinref part="CON_VCC_SWITCH" gate="G$1" pin="2"/>
-<wire x1="-17.78" y1="124.46" x2="-45.72" y2="124.46" width="0.1524" layer="91"/>
-<label x="-45.72" y="124.46" size="1.778" layer="95"/>
+<wire x1="17.78" y1="93.98" x2="45.72" y2="93.98" width="0.1524" layer="91"/>
+<label x="45.72" y="93.98" size="1.778" layer="95" rot="MR0"/>
 </segment>
 <segment>
@@
 <segment>
 <pinref part="CON_REED" gate="G$1" pin="1"/>
-<wire x1="-17.78" y1="111.76" x2="-45.72" y2="111.76" width="0.1524" layer="91"/>
-<label x="-45.72" y="111.76" size="1.778" layer="95"/>
+<wire x1="-43.18" y1="109.22" x2="-15.24" y2="109.22" width="0.1524" layer="91"/>
+<label x="-15.24" y="109.22" size="1.778" layer="95" rot="MR0"/>
 </segment>
 <segment>
@@
 <segment>
 <pinref part="JMP_VCC_COIN_OR_ALT" gate="G$1" pin="3"/>
-<wire x1="-38.1" y1="144.78" x2="-22.86" y2="144.78" width="0.1524" layer="91"/>
-<label x="-35.56" y="144.78" size="1.778" layer="95"/>
+<wire x1="22.86" y1="132.08" x2="38.1" y2="132.08" width="0.1524" layer="91"/>
+<label x="25.4" y="132.08" size="1.778" layer="95"/>
+</segment>
+<segment>
+<pinref part="CON_COIN_HOLDER" gate="G$1" pin="1"/>
+<wire x1="17.78" y1="114.3" x2="30.48" y2="114.3" width="0.1524" layer="91"/>
+<pinref part="C1" gate="G$1" pin="1"/>
+<wire x1="30.48" y1="114.3" x2="38.1" y2="114.3" width="0.1524" layer="91"/>
+<wire x1="38.1" y1="114.3" x2="48.26" y2="114.3" width="0.1524" layer="91"/>
+<junction x="38.1" y="114.3"/>
+<pinref part="C2" gate="G$1" pin="1"/>
+<junction x="30.48" y="114.3"/>
+<label x="48.26" y="114.3" size="1.778" layer="95" rot="MR0"/>
 </segment>
 </net>
@@
 <segment>
 <pinref part="JMP_VCC_COIN_OR_ALT" gate="G$1" pin="1"/>
-<wire x1="-38.1" y1="139.7" x2="-22.86" y2="139.7" width="0.1524" layer="91"/>
-<label x="-35.56" y="139.7" size="1.778" layer="95"/>
-</segment>
-</net>
+<wire x1="22.86" y1="127" x2="38.1" y2="127" width="0.1524" layer="91"/>
+<label x="25.4" y="127" size="1.778" layer="95"/>
+</segment>
+</net>

Commit message: [ add ] main.bom
Parts:
- removed C2: 330u, rcl:C-EUC1206K
- added C3: 330u, rcl:CPOL-EUF
- CON_COIN_HOLDER, CON_REED, CON_VCC_SWITCH: device pinhead:PINHD-1X2 -> SparkFun:M02PTH
- CON_GND, CON_IO, CON_VCC_EN: device con-lstb:MA05-1 -> SparkFun:M05PTH
- JMP_VCC_COIN_OR_ALT: device con-lstb:MA03-1 -> SparkFun:M03PTH
- R1: value 470K -> 1M
Connections:
- net COIN_VCC: now also C3.+; no longer C2.1
- net GND: now also C3.-; no longer C2.2
Other:
- moved on the sheet: C1, CON_COIN_HOLDER, CON_GND, CON_IO, CON_REED, CON_VCC_EN, CON_VCC_SWITCH, JMP_VCC_COIN_OR_ALT
Changed lines of the file:
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@@
 <setting verticaltext="up"/>
 </settings>
-<grid distance="2.54" unitdist="mm" unit="mm" style="lines" multiple="1" display="yes" altdistance="0.01" altunitdist="inch" altunit="inch"/>
+<grid distance="1.27" unitdist="mm" unit="mm" style="lines" multiple="1" display="yes" altdistance="0.01" altunitdist="inch" altunit="inch"/>
 <layers>
 <layer number="1" name="Top" color="4" fill="1" visible="no" active="no"/>
@@
 <part name="CON_NRF" library="con-lstb" deviceset="MA07-2" device=""/>
 <part name="C1" library="rcl" deviceset="C-EU" device="C1206K" value="100n"/>
-<part name="R1" library="resistor" deviceset="R-EU_" device="R1206" value="470K"/>
-<part name="CON_REED" library="pinhead" deviceset="PINHD-1X2" device=""/>
-<part name="CON_GND" library="con-lstb" deviceset="MA05-1" device=""/>
-<part name="CON_VCC_EN" library="con-lstb" deviceset="MA05-1" device=""/>
-<part name="CON_IO" library="con-lstb" deviceset="MA05-1" device=""/>
-<part name="CON_VCC_SWITCH" library="pinhead" deviceset="PINHD-1X2" device=""/>
-<part name="JMP_VCC_COIN_OR_ALT" library="con-lstb" deviceset="MA03-1" device=""/>
-<part name="CON_COIN_HOLDER" library="pinhead" deviceset="PINHD-1X2" device=""/>
-<part name="C2" library="rcl" deviceset="C-EU" device="C1206K" value="330u"/>
+<part name="R1" library="resistor" deviceset="R-EU_" device="R1206" value="1M"/>
+<part name="CON_REED" library="SparkFun" deviceset="M02" device="PTH"/>
+<part name="CON_GND" library="SparkFun" deviceset="M05" device="PTH"/>
+<part name="CON_VCC_EN" library="SparkFun" deviceset="M05" device="PTH"/>
+<part name="CON_IO" library="SparkFun" deviceset="M05" device="PTH"/>
+<part name="CON_VCC_SWITCH" library="SparkFun" deviceset="M02" device="PTH"/>
+<part name="JMP_VCC_COIN_OR_ALT" library="SparkFun" deviceset="M03" device="PTH"/>
+<part name="CON_COIN_HOLDER" library="SparkFun" deviceset="M02" device="PTH"/>
 <part name="FRAME1" library="frames" deviceset="A4L-LOC" device=""/>
+<part name="C3" library="rcl" deviceset="CPOL-EU" device="F" value="330u"/>
 </parts>
 <sheets>
@@
 <instance part="PCB1" gate="G$1" x="30.48" y="58.42" rot="R270"/>
 <instance part="CON_NRF" gate="G$1" x="109.22" y="55.88"/>
-<instance part="C1" gate="G$1" x="38.1" y="111.76" rot="MR0"/>
+<instance part="C1" gate="G$1" x="35.56" y="111.76" smashed="yes" rot="MR0">
+<attribute name="NAME" x="34.036" y="112.141" size="1.778" layer="95" rot="MR0"/>
+<attribute name="VALUE" x="41.656" y="107.061" size="1.778" layer="96" rot="MR0"/>
+</instance>
 <instance part="R1" gate="G$1" x="-33.02" y="106.68" rot="MR0"/>
-<instance part="CON_REED" gate="G$1" x="-45.72" y="106.68" smashed="yes" rot="MR0">
-<attribute name="NAME" x="-34.29" y="112.395" size="1.778" layer="95" rot="MR0"/>
-<attribute name="VALUE" x="-39.37" y="101.6" size="1.778" layer="96" rot="MR0"/>
+<instance part="CON_REED" gate="G$1" x="-45.72" y="109.22" smashed="yes" rot="MR180">
+<attribute name="NAME" x="-46.99" y="114.935" size="1.778" layer="95" rot="MR180"/>
+<attribute name="VALUE" x="-52.07" y="114.3" size="1.778" layer="96" rot="MR180"/>
 </instance>
 <instance part="CON_GND" gate="G$1" x="-45.72" y="40.64"/>
 <instance part="CON_VCC_EN" gate="G$1" x="-45.72" y="63.5"/>
 <instance part="CON_IO" gate="G$1" x="-45.72" y="86.36"/>
-<instance part="CON_VCC_SWITCH" gate="G$1" x="15.24" y="93.98" smashed="yes" rot="MR0">
-<attribute name="NAME" x="36.83" y="99.695" size="1.778" layer="95" rot="MR0"/>
-<attribute name="VALUE" x="21.59" y="88.9" size="1.778" layer="96" rot="MR0"/>
+<instance part="CON_VCC_SWITCH" gate="G$1" x="15.24" y="96.52" smashed="yes" rot="MR180">
+<attribute name="NAME" x="13.97" y="102.235" size="1.778" layer="95" rot="MR180"/>
+<attribute name="VALUE" x="8.89" y="101.6" size="1.778" layer="96" rot="MR180"/>
 </instance>
 <instance part="JMP_VCC_COIN_OR_ALT" gate="G$1" x="15.24" y="129.54"/>
-<instance part="CON_COIN_HOLDER" gate="G$1" x="15.24" y="111.76" smashed="yes" rot="MR0">
-<attribute name="NAME" x="36.83" y="117.475" size="1.778" layer="95" rot="MR0"/>
-<attribute name="VALUE" x="21.59" y="106.68" size="1.778" layer="96" rot="MR0"/>
+<instance part="CON_COIN_HOLDER" gate="G$1" x="15.24" y="114.3" smashed="yes" rot="MR180">
+<attribute name="NAME" x="12.7" y="120.015" size="1.778" layer="95" rot="MR180"/>
+<attribute name="VALUE" x="8.89" y="119.38" size="1.778" layer="96" rot="MR180"/>
 </instance>
-<instance part="C2" gate="G$1" x="30.48" y="111.76" rot="MR0"/>
 <instance part="FRAME1" gate="G$1" x="-99.06" y="-15.24" smashed="yes">
 <attribute name="DRAWING_NAME" x="118.11" y="0" size="2.54" layer="94" font="vector"/>
@@
 <attribute name="SHEET" x="131.445" y="-10.16" size="2.54" layer="94" font="vector"/>
 </instance>
+<instance part="C3" gate="G$1" x="26.67" y="111.76"/>
 </instances>
 <busses>
@@
 <segment>
 <pinref part="CON_COIN_HOLDER" gate="G$1" pin="2"/>
-<wire x1="17.78" y1="111.76" x2="17.78" y2="106.68" width="0.1524" layer="91"/>
-<wire x1="17.78" y1="106.68" x2="30.48" y2="106.68" width="0.1524" layer="91"/>
+<wire x1="22.86" y1="111.76" x2="22.86" y2="106.68" width="0.1524" layer="91"/>
 <label x="48.26" y="106.68" size="1.778" layer="95" rot="MR0"/>
 <pinref part="C1" gate="G$1" pin="2"/>
-<wire x1="30.48" y1="106.68" x2="38.1" y2="106.68" width="0.1524" layer="91"/>
-<wire x1="38.1" y1="106.68" x2="48.26" y2="106.68" width="0.1524" layer="91"/>
-<junction x="38.1" y="106.68"/>
-<pinref part="C2" gate="G$1" pin="2"/>
-<junction x="30.48" y="106.68"/>
+<wire x1="22.86" y1="106.68" x2="26.67" y2="106.68" width="0.1524" layer="91"/>
+<wire x1="26.67" y1="106.68" x2="35.56" y2="106.68" width="0.1524" layer="91"/>
+<wire x1="35.56" y1="106.68" x2="48.26" y2="106.68" width="0.1524" layer="91"/>
+<junction x="35.56" y="106.68"/>
+<pinref part="C3" gate="G$1" pin="-"/>
+<junction x="26.67" y="106.68"/>
 </segment>
 </net>
@@
 <pinref part="CON_REED" gate="G$1" pin="2"/>
 <pinref part="R1" gate="G$1" pin="2"/>
-<wire x1="-43.18" y1="106.68" x2="-38.1" y2="106.68" width="0.1524" layer="91"/>
 <wire x1="-38.1" y1="106.68" x2="-38.1" y2="101.6" width="0.1524" layer="91"/>
 <junction x="-38.1" y="106.68"/>
@@
 <segment>
 <pinref part="CON_VCC_SWITCH" gate="G$1" pin="1"/>
-<wire x1="17.78" y1="96.52" x2="45.72" y2="96.52" width="0.1524" layer="91"/>
+<wire x1="22.86" y1="96.52" x2="45.72" y2="96.52" width="0.1524" layer="91"/>
 <label x="45.72" y="96.52" size="1.778" layer="95" rot="MR0"/>
 </segment>
@@
 <segment>
 <pinref part="CON_VCC_SWITCH" gate="G$1" pin="2"/>
-<wire x1="17.78" y1="93.98" x2="45.72" y2="93.98" width="0.1524" layer="91"/>
+<wire x1="22.86" y1="93.98" x2="45.72" y2="93.98" width="0.1524" layer="91"/>
 <label x="45.72" y="93.98" size="1.778" layer="95" rot="MR0"/>
 </segment>
@@
 <segment>
 <pinref part="CON_REED" gate="G$1" pin="1"/>
-<wire x1="-43.18" y1="109.22" x2="-15.24" y2="109.22" width="0.1524" layer="91"/>
+<wire x1="-38.1" y1="109.22" x2="-15.24" y2="109.22" width="0.1524" layer="91"/>
 <label x="-15.24" y="109.22" size="1.778" layer="95" rot="MR0"/>
 </segment>
@@
 <segment>
 <pinref part="CON_COIN_HOLDER" gate="G$1" pin="1"/>
-<wire x1="17.78" y1="114.3" x2="30.48" y2="114.3" width="0.1524" layer="91"/>
 <pinref part="C1" gate="G$1" pin="1"/>
-<wire x1="30.48" y1="114.3" x2="38.1" y2="114.3" width="0.1524" layer="91"/>
-<wire x1="38.1" y1="114.3" x2="48.26" y2="114.3" width="0.1524" layer="91"/>
-<junction x="38.1" y="114.3"/>
-<pinref part="C2" gate="G$1" pin="1"/>
-<junction x="30.48" y="114.3"/>
+<wire x1="22.86" y1="114.3" x2="26.67" y2="114.3" width="0.1524" layer="91"/>
+<wire x1="26.67" y1="114.3" x2="35.56" y2="114.3" width="0.1524" layer="91"/>
+<wire x1="35.56" y1="114.3" x2="48.26" y2="114.3" width="0.1524" layer="91"/>
+<junction x="35.56" y="114.3"/>
 <label x="48.26" y="114.3" size="1.778" layer="95" rot="MR0"/>
-</segment>
-</net>
+<pinref part="C3" gate="G$1" pin="+"/>
+<junction x="26.67" y="114.3"/>
+</segment>
+</net>

Commit message: [ update ] route, wip
Parts:
- removed CON_GND, CON_IO, CON_VCC_EN: (no value), SparkFun:M05PTH
- added GND, IO, VCC: (no value), SparkFun:M04PTH
- CON_COIN_HOLDER: device SparkFun:M02PTH -> SparkFun:BATTERY20PTH
- renumbered CON_NRF to NRF, CON_REED to REED, CON_VCC_SWITCH to VCC_SWITCH, JMP_VCC_COIN_OR_ALT to COIN_OR_ALT
Connections:
- removed net N$9: CON_GND.2
- removed net UC_PORTB1: CON_IO.5, PCB1.9
- net COIN_VCC: now also CON_COIN_HOLDER.+; no longer CON_COIN_HOLDER.1
- net GND: now also CON_COIN_HOLDER.-, GND.1, GND.2, GND.3, GND.4; no longer CON_COIN_HOLDER.2, CON_GND.1, CON_GND.3, CON_GND.4, CON_GND.5
- net POW_VCC_EN: now also VCC.1, VCC.2, VCC.3, VCC.4; no longer CON_VCC_EN.1, CON_VCC_EN.2, CON_VCC_EN.3, CON_VCC_EN.4, CON_VCC_EN.5
- net UC_PORTC0: now also IO.4; no longer CON_IO.4
- net UC_PORTC1: now also IO.3; no longer CON_IO.3
- net UC_PORTC2: now also IO.2; no longer CON_IO.2
- net UC_PORTC3: now also IO.1; no longer CON_IO.1

Commit message: [ add ] board routing, done
Parts:
- removed CON_COIN_HOLDER: (no value), SparkFun:BATTERY20PTH
- added U$1: KEYSTONE_1025_7, keystone_1025_7:KEYSTONE_1025_7
Connections:
- net COIN_VCC: now also U$1.COIN_PLUS; no longer CON_COIN_HOLDER.+
- net GND: now also U$1.COIN_MINUS; no longer CON_COIN_HOLDER.-
Changed lines of the file:
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@@
 <setting verticaltext="up"/>
 </settings>
-<grid distance="0.1" unitdist="inch" unit="inch" style="lines" multiple="1" display="yes" altdistance="0.01" altunitdist="inch" altunit="inch"/>
+<grid distance="0.05" unitdist="inch" unit="inch" style="lines" multiple="1" display="yes" altdistance="0.01" altunitdist="inch" altunit="inch"/>
 <layers>
 <layer number="1" name="Top" color="4" fill="1" visible="no" active="no"/>
@@
 <part name="FRAME1" library="frames" deviceset="A4L-LOC" device=""/>
 <part name="C3" library="rcl" deviceset="CPOL-EU" device="F" value="330u"/>
-<part name="CON_COIN_HOLDER" library="SparkFun" deviceset="BATTERY" device="20PTH"/>
+<part name="U$1" library="keystone_1025_7" deviceset="KEYSTONE_1025_7" device=""/>
 </parts>
 <sheets>
@@
 </instance>
 <instance part="C3" gate="G$1" x="26.67" y="111.76"/>
-<instance part="CON_COIN_HOLDER" gate="G$1" x="17.78" y="114.3" smashed="yes" rot="R180">
-<attribute name="NAME" x="36.83" y="120.65" size="1.778" layer="95" rot="R180"/>
-<attribute name="VALUE" x="21.59" y="120.65" size="1.778" layer="96" rot="R180"/>
-</instance>
+<instance part="U$1" gate="G$1" x="17.78" y="114.3"/>
 </instances>
 <busses>
@@
 <pinref part="C3" gate="G$1" pin="-"/>
 <junction x="26.67" y="106.68"/>
-<pinref part="CON_COIN_HOLDER" gate="G$1" pin="-"/>
 <wire x1="12.7" y1="114.3" x2="12.7" y2="106.68" width="0.1524" layer="91"/>
+<wire x1="12.7" y1="114.3" x2="13.97" y2="114.3" width="0.1524" layer="91"/>
+<pinref part="U$1" gate="G$1" pin="COIN_MINUS"/>
 </segment>
 <segment>
@@
 <label x="48.26" y="114.3" size="1.778" layer="95" rot="MR0"/>
 <pinref part="C3" gate="G$1" pin="+"/>
-<pinref part="CON_COIN_HOLDER" gate="G$1" pin="+"/>
-<wire x1="26.67" y1="114.3" x2="22.86" y2="114.3" width="0.1524" layer="91"/>
+<wire x1="26.67" y1="114.3" x2="21.59" y2="114.3" width="0.1524" layer="91"/>
 <junction x="26.67" y="114.3"/>
-</segment>
-</net>
+<pinref part="U$1" gate="G$1" pin="COIN_PLUS"/>
+</segment>
+</net>
